File: Power_Distribution_Board/Power_Distribution_Board.kicad_pcb (KiCad board)
At the start: 2 copper layers, 180 x 165 mm, 50 parts, among them J1 XT60PW-F, J10 XT60PW-F, J11 XT60PW-F, J12 XT60PW-F, J13 XT60PW-F, J14 XT60PW-F, J15 XT30PW-F, J16 XT30PW-F, J17 XT30PW-F, J18 XT30PW-F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

Commit message: Buck changed
Parts:
- removed J5: DCM3623T75H26C2T00, URC_Active:DCM3623T75H26C2T00
- added H11: MountingHole_Pad, MountingHole:MountingHole_3.2mm_M3_Pad, F.Cu at (85.0, 121.0)
- added PS4: PKJ7216ZWPI, URC_Active:PKJ7216ZWPI, B.Cu at (127.4, 180.3)
- J1, J10, J11, J12, J13, J14, J2, J21, J22, J23, J24, J25, J26, J27, J3, J4, J6, J7, J8, J9: footprint URC_Con:XT60PWF -> URC_Conn:XT60PWF
- J15, J16, J17, J18, J19, J20: footprint URC_Con:XT30PWF -> URC_Conn:XT30PWF
- PS1: footprint URC_Con:XT60PWM -> URC_Conn:XT60PWM
- moved H9 92.4 mm to (85.0, 80.5)
- moved H10 90.4 mm to (123.0, 121.0)
- moved H6 78.7 mm to (160.5, 88.5)
- moved H7 78.7 mm to (160.5, 176.5)
- moved H5 72.5 mm to (206.5, 88.5)
- moved H8 58.1 mm to (206.5, 176.5)
- moved PS3 2.04 mm to (128.1, 82.7)
- moved PS2 1.18 mm to (136.8, 103.5)
